Commit message: robot urdf modification, added roller links, switched gz sim to run without gui for better performance, finaly gz plugin ie. omni drive

File: ros_gz_omni_description/models/omni_drive/robot.urdf (robot description, URDF)
Before this commit: robot omni_drive, 10 links, 9 joints
Links:
- removed link wheel_4
- removed link wheel_4_2
- removed link wheel_4_3
- removed link wheel_4_4
- added link wheel4_omniwheel_tyre_v1, mass 0.00502735; collision mesh filename=package://meshes/wheel4_omniwheel_tyre_v1.stl; visual mesh filename=package://meshes/wheel4_omniwheel_tyre_v1.stl
- added link wheel4_omniwheel_tyre_v1_10, mass 0.00502735; collision mesh filename=package://meshes/wheel4_omniwheel_tyre_v1.stl; visual mesh filename=package://meshes/wheel4_omniwheel_tyre_v1.stl
- added link wheel4_omniwheel_tyre_v1_11, mass 0.00502735; collision mesh filename=package://meshes/wheel4_omniwheel_tyre_v1.stl; visual mesh filename=package://meshes/wheel4_omniwheel_tyre_v1.stl
- added link wheel4_omniwheel_tyre_v1_12, mass 0.00502735; collision mesh filename=package://meshes/wheel4_omniwheel_tyre_v1.stl; visual mesh filename=package://meshes/wheel4_omniwheel_tyre_v1.stl
- added link wheel4_omniwheel_tyre_v1_13, mass 0.00502735; collision mesh filename=package://meshes/wheel4_omniwheel_tyre_v1.stl; visual mesh filename=package://meshes/wheel4_omniwheel_tyre_v1.stl
- added link wheel4_omniwheel_tyre_v1_14, mass 0.00502735; collision mesh filename=package://meshes/wheel4_omniwheel_tyre_v1.stl; visual mesh filename=package://meshes/wheel4_omniwheel_tyre_v1.stl
- added link wheel4_omniwheel_tyre_v1_15, mass 0.00502735; collision mesh filename=package://meshes/wheel4_omniwheel_tyre_v1.stl; visual mesh filename=package://meshes/wheel4_omniwheel_tyre_v1.stl
- added link wheel4_omniwheel_tyre_v1_16, mass 0.00502735; collision mesh filename=package://meshes/wheel4_omniwheel_tyre_v1.stl; visual mesh filename=package://meshes/wheel4_omniwheel_tyre_v1.stl
- added link wheel4_omniwheel_tyre_v1_17, mass 0.00502735; collision mesh filename=package://meshes/wheel4_omniwheel_tyre_v1.stl; visual mesh filename=package://meshes/wheel4_omniwheel_tyre_v1.stl
- added link wheel4_omniwheel_tyre_v1_18, mass 0.00502735; collision mesh filename=package://meshes/wheel4_omniwheel_tyre_v1.stl; visual mesh filename=package://meshes/wheel4_omniwheel_tyre_v1.stl
- added link wheel4_omniwheel_tyre_v1_19, mass 0.00502735; collision mesh filename=package://meshes/wheel4_omniwheel_tyre_v1.stl; visual mesh filename=package://meshes/wheel4_omniwheel_tyre_v1.stl
- added link wheel4_omniwheel_tyre_v1_2, mass 0.00502735; collision mesh filename=package://meshes/wheel4_omniwheel_tyre_v1.stl; visual mesh filename=package://meshes/wheel4_omniwheel_tyre_v1.stl
- added link wheel4_omniwheel_tyre_v1_20, mass 0.00502735; collision mesh filename=package://meshes/wheel4_omniwheel_tyre_v1.stl; visual mesh filename=package://meshes/wheel4_omniwheel_tyre_v1.stl
- added link wheel4_omniwheel_tyre_v1_21, mass 0.00502735; collision mesh filename=package://meshes/wheel4_omniwheel_tyre_v1.stl; visual mesh filename=package://meshes/wheel4_omniwheel_tyre_v1.stl
- added link wheel4_omniwheel_tyre_v1_22, mass 0.00502735; collision mesh filename=package://meshes/wheel4_omniwheel_tyre_v1.stl; visual mesh filename=package://meshes/wheel4_omniwheel_tyre_v1.stl
- added link wheel4_omniwheel_tyre_v1_23, mass 0.00502735; collision mesh filename=package://meshes/wheel4_omniwheel_tyre_v1.stl; visual mesh filename=package://meshes/wheel4_omniwheel_tyre_v1.stl
- added link wheel4_omniwheel_tyre_v1_24, mass 0.00502735; collision mesh filename=package://meshes/wheel4_omniwheel_tyre_v1.stl; visual mesh filename=package://meshes/wheel4_omniwheel_tyre_v1.stl
- added link wheel4_omniwheel_tyre_v1_25, mass 0.00502735; collision mesh filename=package://meshes/wheel4_omniwheel_tyre_v1.stl; visual mesh filename=package://meshes/wheel4_omniwheel_tyre_v1.stl
- added link wheel4_omniwheel_tyre_v1_26, mass 0.00502735; collision mesh filename=package://meshes/wheel4_omniwheel_tyre_v1.stl; visual mesh filename=package://meshes/wheel4_omniwheel_tyre_v1.stl
- added link wheel4_omniwheel_tyre_v1_27, mass 0.00502735; collision mesh filename=package://meshes/wheel4_omniwheel_tyre_v1.stl; visual mesh filename=package://meshes/wheel4_omniwheel_tyre_v1.stl
- added link wheel4_omniwheel_tyre_v1_28, mass 0.00502735; collision mesh filename=package://meshes/wheel4_omniwheel_tyre_v1.stl; visual mesh filename=package://meshes/wheel4_omniwheel_tyre_v1.stl
- added link wheel4_omniwheel_tyre_v1_29, mass 0.00502735; collision mesh filename=package://meshes/wheel4_omniwheel_tyre_v1.stl; visual mesh filename=package://meshes/wheel4_omniwheel_tyre_v1.stl
- added link wheel4_omniwheel_tyre_v1_3, mass 0.00502735; collision mesh filename=package://meshes/wheel4_omniwheel_tyre_v1.stl; visual mesh filename=package://meshes/wheel4_omniwheel_tyre_v1.stl
- added link wheel4_omniwheel_tyre_v1_30, mass 0.00502735; collision mesh filename=package://meshes/wheel4_omniwheel_tyre_v1.stl; visual mesh filename=package://meshes/wheel4_omniwheel_tyre_v1.stl
- added link wheel4_omniwheel_tyre_v1_31, mass 0.00502735; collision mesh filename=package://meshes/wheel4_omniwheel_tyre_v1.stl; visual mesh filename=package://meshes/wheel4_omniwheel_tyre_v1.stl
- added link wheel4_omniwheel_tyre_v1_32, mass 0.00502735; collision mesh filename=package://meshes/wheel4_omniwheel_tyre_v1.stl; visual mesh filename=package://meshes/wheel4_omniwheel_tyre_v1.stl
- added link wheel4_omniwheel_tyre_v1_33, mass 0.00502735; collision mesh filename=package://meshes/wheel4_omniwheel_tyre_v1.stl; visual mesh filename=package://meshes/wheel4_omniwheel_tyre_v1.stl
- added link wheel4_omniwheel_tyre_v1_34, mass 0.00502735; collision mesh filename=package://meshes/wheel4_omniwheel_tyre_v1.stl; visual mesh filename=package://meshes/wheel4_omniwheel_tyre_v1.stl
- added link wheel4_omniwheel_tyre_v1_35, mass 0.00502735; collision mesh filename=package://meshes/wheel4_omniwheel_tyre_v1.stl; visual mesh filename=package://meshes/wheel4_omniwheel_tyre_v1.stl
- added link wheel4_omniwheel_tyre_v1_36, mass 0.00502735; collision mesh filename=package://meshes/wheel4_omniwheel_tyre_v1.stl; visual mesh filename=package://meshes/wheel4_omniwheel_tyre_v1.stl
- added link wheel4_omniwheel_tyre_v1_37, mass 0.00502735; collision mesh filename=package://meshes/wheel4_omniwheel_tyre_v1.stl; visual mesh filename=package://meshes/wheel4_omniwheel_tyre_v1.stl
- added link wheel4_omniwheel_tyre_v1_38, mass 0.00502735; collision mesh filename=package://meshes/wheel4_omniwheel_tyre_v1.stl; visual mesh filename=package://meshes/wheel4_omniwheel_tyre_v1.stl
- added link wheel4_omniwheel_tyre_v1_39, mass 0.00502735; collision mesh filename=package://meshes/wheel4_omniwheel_tyre_v1.stl; visual mesh filename=package://meshes/wheel4_omniwheel_tyre_v1.stl
- added link wheel4_omniwheel_tyre_v1_4, mass 0.00502735; collision mesh filename=package://meshes/wheel4_omniwheel_tyre_v1.stl; visual mesh filename=package://meshes/wheel4_omniwheel_tyre_v1.stl
- added link wheel4_omniwheel_tyre_v1_40, mass 0.00502735; collision mesh filename=package://meshes/wheel4_omniwheel_tyre_v1.stl; visual mesh filename=package://meshes/wheel4_omniwheel_tyre_v1.stl
- added link wheel4_omniwheel_tyre_v1_41, mass 0.00502735; collision mesh filename=package://meshes/wheel4_omniwheel_tyre_v1.stl; visual mesh filename=package://meshes/wheel4_omniwheel_tyre_v1.stl
- added link wheel4_omniwheel_tyre_v1_42, mass 0.00502735; collision mesh filename=package://meshes/wheel4_omniwheel_tyre_v1.stl; visual mesh filename=package://meshes/wheel4_omniwheel_tyre_v1.stl
- added link wheel4_omniwheel_tyre_v1_43, mass 0.00502735; collision mesh filename=package://meshes/wheel4_omniwheel_tyre_v1.stl; visual mesh filename=package://meshes/wheel4_omniwheel_tyre_v1.stl
- added link wheel4_omniwheel_tyre_v1_44, mass 0.00502735; collision mesh filename=package://meshes/wheel4_omniwheel_tyre_v1.stl; visual mesh filename=package://meshes/wheel4_omniwheel_tyre_v1.stl
- added link wheel4_omniwheel_tyre_v1_45, mass 0.00502735; collision mesh filename=package://meshes/wheel4_omniwheel_tyre_v1.stl; visual mesh filename=package://meshes/wheel4_omniwheel_tyre_v1.stl
- added link wheel4_omniwheel_tyre_v1_46, mass 0.00502735; collision mesh filename=package://meshes/wheel4_omniwheel_tyre_v1.stl; visual mesh filename=package://meshes/wheel4_omniwheel_tyre_v1.stl
- added link wheel4_omniwheel_tyre_v1_47, mass 0.00502735; collision mesh filename=package://meshes/wheel4_omniwheel_tyre_v1.stl; visual mesh filename=package://meshes/wheel4_omniwheel_tyre_v1.stl
- added link wheel4_omniwheel_tyre_v1_48, mass 0.00502735; collision mesh filename=package://meshes/wheel4_omniwheel_tyre_v1.stl; visual mesh filename=package://meshes/wheel4_omniwheel_tyre_v1.stl
- added link wheel4_omniwheel_tyre_v1_49, mass 0.00502735; collision mesh filename=package://meshes/wheel4_omniwheel_tyre_v1.stl; visual mesh filename=package://meshes/wheel4_omniwheel_tyre_v1.stl
- added link wheel4_omniwheel_tyre_v1_5, mass 0.00502735; collision mesh filename=package://meshes/wheel4_omniwheel_tyre_v1.stl; visual mesh filename=package://meshes/wheel4_omniwheel_tyre_v1.stl
- added link wheel4_omniwheel_tyre_v1_50, mass 0.00502735; collision mesh filename=package://meshes/wheel4_omniwheel_tyre_v1.stl; visual mesh filename=package://meshes/wheel4_omniwheel_tyre_v1.stl
- added link wheel4_omniwheel_tyre_v1_51, mass 0.00502735; collision mesh filename=package://meshes/wheel4_omniwheel_tyre_v1.stl; visual mesh filename=package://meshes/wheel4_omniwheel_tyre_v1.stl
- added link wheel4_omniwheel_tyre_v1_52, mass 0.00502735; collision mesh filename=package://meshes/wheel4_omniwheel_tyre_v1.stl; visual mesh filename=package://meshes/wheel4_omniwheel_tyre_v1.stl
- added link wheel4_omniwheel_tyre_v1_53, mass 0.00502735; collision mesh filename=package://meshes/wheel4_omniwheel_tyre_v1.stl; visual mesh filename=package://meshes/wheel4_omniwheel_tyre_v1.stl
- added link wheel4_omniwheel_tyre_v1_54, mass 0.00502735; collision mesh filename=package://meshes/wheel4_omniwheel_tyre_v1.stl; visual mesh filename=package://meshes/wheel4_omniwheel_tyre_v1.stl
- added link wheel4_omniwheel_tyre_v1_55, mass 0.00502735; collision mesh filename=package://meshes/wheel4_omniwheel_tyre_v1.stl; visual mesh filename=package://meshes/wheel4_omniwheel_tyre_v1.stl
- added link wheel4_omniwheel_tyre_v1_56, mass 0.00502735; collision mesh filename=package://meshes/wheel4_omniwheel_tyre_v1.stl; visual mesh filename=package://meshes/wheel4_omniwheel_tyre_v1.stl
- added link wheel4_omniwheel_tyre_v1_57, mass 0.00502735; collision mesh filename=package://meshes/wheel4_omniwheel_tyre_v1.stl; visual mesh filename=package://meshes/wheel4_omniwheel_tyre_v1.stl
- added link wheel4_omniwheel_tyre_v1_58, mass 0.00502735; collision mesh filename=package://meshes/wheel4_omniwheel_tyre_v1.stl; visual mesh filename=package://meshes/wheel4_omniwheel_tyre_v1.stl
- added link wheel4_omniwheel_tyre_v1_59, mass 0.00502735; collision mesh filename=package://meshes/wheel4_omniwheel_tyre_v1.stl; visual mesh filename=package://meshes/wheel4_omniwheel_tyre_v1.stl
- added link wheel4_omniwheel_tyre_v1_6, mass 0.00502735; collision mesh filename=package://meshes/wheel4_omniwheel_tyre_v1.stl; visual mesh filename=package://meshes/wheel4_omniwheel_tyre_v1.stl
- added link wheel4_omniwheel_tyre_v1_60, mass 0.00502735; collision mesh filename=package://meshes/wheel4_omniwheel_tyre_v1.stl; visual mesh filename=package://meshes/wheel4_omniwheel_tyre_v1.stl
- added link wheel4_omniwheel_tyre_v1_61, mass 0.00502735; collision mesh filename=package://meshes/wheel4_omniwheel_tyre_v1.stl; visual mesh filename=package://meshes/wheel4_omniwheel_tyre_v1.stl
- added link wheel4_omniwheel_tyre_v1_62, mass 0.00502735; collision mesh filename=package://meshes/wheel4_omniwheel_tyre_v1.stl; visual mesh filename=package://meshes/wheel4_omniwheel_tyre_v1.stl
- added link wheel4_omniwheel_tyre_v1_63, mass 0.00502735; collision mesh filename=package://meshes/wheel4_omniwheel_tyre_v1.stl; visual mesh filename=package://meshes/wheel4_omniwheel_tyre_v1.stl
- added link wheel4_omniwheel_tyre_v1_64, mass 0.00502735; collision mesh filename=package://meshes/wheel4_omniwheel_tyre_v1.stl; visual mesh filename=package://meshes/wheel4_omniwheel_tyre_v1.stl
- added link wheel4_omniwheel_tyre_v1_65, mass 0.00502735; collision mesh filename=package://meshes/wheel4_omniwheel_tyre_v1.stl; visual mesh filename=package://meshes/wheel4_omniwheel_tyre_v1.stl
- added link wheel4_omniwheel_tyre_v1_66, mass 0.00502735; collision mesh filename=package://meshes/wheel4_omniwheel_tyre_v1.stl; visual mesh filename=package://meshes/wheel4_omniwheel_tyre_v1.stl
- added link wheel4_omniwheel_tyre_v1_67, mass 0.00502735; collision mesh filename=package://meshes/wheel4_omniwheel_tyre_v1.stl; visual mesh filename=package://meshes/wheel4_omniwheel_tyre_v1.stl
- added link wheel4_omniwheel_tyre_v1_68, mass 0.00502735; collision mesh filename=package://meshes/wheel4_omniwheel_tyre_v1.stl; visual mesh filename=package://meshes/wheel4_omniwheel_tyre_v1.stl
- added link wheel4_omniwheel_tyre_v1_69, mass 0.00502735; collision mesh filename=package://meshes/wheel4_omniwheel_tyre_v1.stl; visual mesh filename=package://meshes/wheel4_omniwheel_tyre_v1.stl
- added link wheel4_omniwheel_tyre_v1_7, mass 0.00502735; collision mesh filename=package://meshes/wheel4_omniwheel_tyre_v1.stl; visual mesh filename=package://meshes/wheel4_omniwheel_tyre_v1.stl
- added link wheel4_omniwheel_tyre_v1_70, mass 0.00502735; collision mesh filename=package://meshes/wheel4_omniwheel_tyre_v1.stl; visual mesh filename=package://meshes/wheel4_omniwheel_tyre_v1.stl
- added link wheel4_omniwheel_tyre_v1_71, mass 0.00502735; collision mesh filename=package://meshes/wheel4_omniwheel_tyre_v1.stl; visual mesh filename=package://meshes/wheel4_omniwheel_tyre_v1.stl
- added link wheel4_omniwheel_tyre_v1_72, mass 0.00502735; collision mesh filename=package://meshes/wheel4_omniwheel_tyre_v1.stl; visual mesh filename=package://meshes/wheel4_omniwheel_tyre_v1.stl
- added link wheel4_omniwheel_tyre_v1_73, mass 0.00502735; collision mesh filename=package://meshes/wheel4_omniwheel_tyre_v1.stl; visual mesh filename=package://meshes/wheel4_omniwheel_tyre_v1.stl
- added link wheel4_omniwheel_tyre_v1_74, mass 0.00502735; collision mesh filename=package://meshes/wheel4_omniwheel_tyre_v1.stl; visual mesh filename=package://meshes/wheel4_omniwheel_tyre_v1.stl
- added link wheel4_omniwheel_tyre_v1_75, mass 0.00502735; collision mesh filename=package://meshes/wheel4_omniwheel_tyre_v1.stl; visual mesh filename=package://meshes/wheel4_omniwheel_tyre_v1.stl
- added link wheel4_omniwheel_tyre_v1_76, mass 0.00502735; collision mesh filename=package://meshes/wheel4_omniwheel_tyre_v1.stl; visual mesh filename=package://meshes/wheel4_omniwheel_tyre_v1.stl
- added link wheel4_omniwheel_tyre_v1_77, mass 0.00502735; collision mesh filename=package://meshes/wheel4_omniwheel_tyre_v1.stl; visual mesh filename=package://meshes/wheel4_omniwheel_tyre_v1.stl
- added link wheel4_omniwheel_tyre_v1_78, mass 0.00502735; collision mesh filename=package://meshes/wheel4_omniwheel_tyre_v1.stl; visual mesh filename=package://meshes/wheel4_omniwheel_tyre_v1.stl
- added link wheel4_omniwheel_tyre_v1_79, mass 0.00502735; collision mesh filename=package://meshes/wheel4_omniwheel_tyre_v1.stl; visual mesh filename=package://meshes/wheel4_omniwheel_tyre_v1.stl
- added link wheel4_omniwheel_tyre_v1_8, mass 0.00502735; collision mesh filename=package://meshes/wheel4_omniwheel_tyre_v1.stl; visual mesh filename=package://meshes/wheel4_omniwheel_tyre_v1.stl
- added link wheel4_omniwheel_tyre_v1_80, mass 0.00502735; collision mesh filename=package://meshes/wheel4_omniwheel_tyre_v1.stl; visual mesh filename=package://meshes/wheel4_omniwheel_tyre_v1.stl
- added link wheel4_omniwheel_tyre_v1_9, mass 0.00502735; collision mesh filename=package://meshes/wheel4_omniwheel_tyre_v1.stl; visual mesh filename=package://meshes/wheel4_omniwheel_tyre_v1.stl
- added link wheel4_shaft_holder_v2, mass 0.162524; visual mesh filename=package://meshes/wheel4_body_omni_v4.stl; visual mesh filename=package://meshes/wheel4_body_omni_v4__2.stl
- added link wheel4_shaft_holder_v2_2, mass 0.162524; visual mesh filename=package://meshes/wheel4_body_omni_v4.stl; visual mesh filename=package://meshes/wheel4_body_omni_v4__2.stl
- added link wheel4_shaft_holder_v2_3, mass 0.162524; visual mesh filename=package://meshes/wheel4_body_omni_v4.stl; visual mesh filename=package://meshes/wheel4_body_omni_v4__2.stl
- added link wheel4_shaft_holder_v2_4, mass 0.162524; visual mesh filename=package://meshes/wheel4_body_omni_v4.stl; visual mesh filename=package://meshes/wheel4_body_omni_v4__2.stl
Joints:
- added joint wheel_2a: type continuous, parent wheel4_shaft_holder_v2_4, child wheel4_omniwheel_tyre_v1_80, origin xyz=0.0384102 -0.0124802 0.0065 rpy=-1.25664 1.5708 0, axis 0 0 1, limit effort=5 velocity=10
- added joint wheel_2b: type continuous, parent wheel4_shaft_holder_v2_4, child wheel4_omniwheel_tyre_v1_79, origin xyz=0.0237388 -0.0326737 0.0065 rpy=-2.51327 -1.5708 0, axis 0 0 1, limit effort=5 velocity=10
- added joint wheel_2c: type continuous, parent wheel4_shaft_holder_v2_4, child wheel4_omniwheel_tyre_v1_78, origin xyz=1.21431e-17 -0.0403869 0.0065 rpy=-3.14159 -1.5708 0, axis 0 0 1, limit effort=5 velocity=10
- added joint wheel_2d: type continuous, parent wheel4_shaft_holder_v2_4, child wheel4_omniwheel_tyre_v1_77, origin xyz=-0.0237388 -0.0326737 0.0065 rpy=1.5708 -1.54071 0.942478, axis 0 0 1, limit effort=5 velocity=10
- added joint wheel_2e: type continuous, parent wheel4_shaft_holder_v2_4, child wheel4_omniwheel_tyre_v1_76, origin xyz=-0.0384102 -0.0124802 0.0065 rpy=1.88496 -1.5708 0, axis 0 0 1, limit effort=5 velocity=10
- added joint wheel_2f: type continuous, parent wheel4_shaft_holder_v2_4, child wheel4_omniwheel_tyre_v1_75, origin xyz=-0.0384102 0.0124802 0.0065 rpy=1.5708 -1.54666 2.82743, axis 0 0 1, limit effort=5 velocity=10
- added joint wheel_2g: type continuous, parent wheel4_shaft_holder_v2_4, child wheel4_omniwheel_tyre_v1_74, origin xyz=-0.0237388 0.0326737 0.0065 rpy=-2.51327 -1.5708 0, axis 0 0 1, limit effort=5 velocity=10
- added joint wheel_2h: type continuous, parent wheel4_shaft_holder_v2_4, child wheel4_omniwheel_tyre_v1_73, origin xyz=1.73472e-18 0.0403869 0.0065 rpy=-4.44089e-16 1.5708 0, axis 0 0 1, limit effort=5 velocity=10
- added joint wheel_2i: type continuous, parent wheel4_shaft_holder_v2_4, child wheel4_omniwheel_tyre_v1_72, origin xyz=0.0237388 0.0326737 0.0065 rpy=2.51327 -1.5708 0, axis 0 0 1, limit effort=5 velocity=10
- added joint wheel_2j: type continuous, parent wheel4_shaft_holder_v2_4, child wheel4_omniwheel_tyre_v1_71, origin xyz=0.0384102 0.0124802 0.0065 rpy=-1.25664 -1.5708 0, axis 0 0 1, limit effort=5 velocity=10
- added joint wheel_2k: type continuous, parent wheel4_shaft_holder_v2_4, child wheel4_omniwheel_tyre_v1_61, origin xyz=-0.0403869 -2.71773e-17 0.0255 rpy=1.5708 0.992087 3.14159, axis 0 0 1, limit effort=5 velocity=10
- added joint wheel_2l: type continuous, parent wheel4_shaft_holder_v2_4, child wheel4_omniwheel_tyre_v1_62, origin xyz=-0.0326737 0.0237388 0.0255 rpy=-2.19911 -1.5708 0, axis 0 0 1, limit effort=5 velocity=10
- added joint wheel_2m: type continuous, parent wheel4_shaft_holder_v2_4, child wheel4_omniwheel_tyre_v1_63, origin xyz=-0.0124802 0.0384102 0.0255 rpy=-2.82743 -1.5708 0, axis 0 0 1, limit effort=5 velocity=10
- added joint wheel_2n: type continuous, parent wheel4_shaft_holder_v2_4, child wheel4_omniwheel_tyre_v1_64, origin xyz=0.0124802 0.0384102 0.0255 rpy=-0.314159 -1.5708 0, axis 0 0 1, limit effort=5 velocity=10
- added joint wheel_2o: type continuous, parent wheel4_shaft_holder_v2_4, child wheel4_omniwheel_tyre_v1_65, origin xyz=0.0326737 0.0237388 0.0255 rpy=-0.942478 -1.5708 0, axis 0 0 1, limit effort=5 velocity=10
- added joint wheel_2p: type continuous, parent wheel4_shaft_holder_v2_4, child wheel4_omniwheel_tyre_v1_66, origin xyz=0.0403869 2.83338e-17 0.0255 rpy=1.5708 0.992087 3.14159, axis 0 0 1, limit effort=5 velocity=10
- added joint wheel_2q: type continuous, parent wheel4_shaft_holder_v2_4, child wheel4_omniwheel_tyre_v1_67, origin xyz=0.0326737 -0.0237388 0.0255 rpy=-2.19911 -1.5708 0, axis 0 0 1, limit effort=5 velocity=10
- added joint wheel_2r: type continuous, parent wheel4_shaft_holder_v2_4, child wheel4_omniwheel_tyre_v1_68, origin xyz=0.0124802 -0.0384102 0.0255 rpy=1.5708 -1.00644 1.88496, axis 0 0 1, limit effort=5 velocity=10
- added joint wheel_2s: type continuous, parent wheel4_shaft_holder_v2_4, child wheel4_omniwheel_tyre_v1_69, origin xyz=-0.0124802 -0.0384102 0.0255 rpy=-0.314159 -1.5708 0, axis 0 0 1, limit effort=5 velocity=10
- added joint wheel_2t: type continuous, parent wheel4_shaft_holder_v2_4, child wheel4_omniwheel_tyre_v1_70, origin xyz=-0.0326737 -0.0237388 0.0255 rpy=-0.942478 -1.5708 0, axis 0 0 1, limit effort=5 velocity=10
- added joint wheel_3a: type continuous, parent wheel4_shaft_holder_v2, child wheel4_omniwheel_tyre_v1_20, origin xyz=0.0384102 -0.0124802 0.0065 rpy=-1.25664 1.5708 0, axis 0 0 1, limit effort=5 velocity=10
- added joint wheel_3b: type continuous, parent wheel4_shaft_holder_v2, child wheel4_omniwheel_tyre_v1_19, origin xyz=0.0237388 -0.0326737 0.0065 rpy=-1.5708 -0.210366 -0.942478, axis 0 0 1, limit effort=5 velocity=10
- added joint wheel_3c: type continuous, parent wheel4_shaft_holder_v2, child wheel4_omniwheel_tyre_v1_18, origin xyz=-3.46945e-18 -0.0403869 0.0065 rpy=-1.5708 -6.10623e-16 -1.5708, axis 0 0 1, limit effort=5 velocity=10
- added joint wheel_3d: type continuous, parent wheel4_shaft_holder_v2, child wheel4_omniwheel_tyre_v1_17, origin xyz=-0.0237388 -0.0326737 0.0065 rpy=-1.5708 -0.240455 -2.19911, axis 0 0 1, limit effort=5 velocity=10
- added joint wheel_3e: type continuous, parent wheel4_shaft_holder_v2, child wheel4_omniwheel_tyre_v1_16, origin xyz=-0.0384102 -0.0124802 0.0065 rpy=-1.5708 -0.971379 -2.82743, axis 0 0 1, limit effort=5 velocity=10
- added joint wheel_3f: type continuous, parent wheel4_shaft_holder_v2, child wheel4_omniwheel_tyre_v1_15, origin xyz=-0.0384102 0.0124802 0.0065 rpy=-1.5708 -0.990694 -0.314159, axis 0 0 1, limit effort=5 velocity=10
- added joint wheel_3g: type continuous, parent wheel4_shaft_holder_v2, child wheel4_omniwheel_tyre_v1_14, origin xyz=-0.0237388 0.0326737 0.0065 rpy=-1.5708 -0.210366 -0.942478, axis 0 0 1, limit effort=5 velocity=10
- added joint wheel_3h: type continuous, parent wheel4_shaft_holder_v2, child wheel4_omniwheel_tyre_v1_13, origin xyz=0 0.0403869 0.0065 rpy=-4.44089e-16 1.5708 0, axis 0 0 1, limit effort=5 velocity=10
- added joint wheel_3i: type continuous, parent wheel4_shaft_holder_v2, child wheel4_omniwheel_tyre_v1_12, origin xyz=0.0237388 0.0326737 0.0065 rpy=-1.5708 -0.210366 -2.19911, axis 0 0 1, limit effort=5 velocity=10
- added joint wheel_3j: type continuous, parent wheel4_shaft_holder_v2, child wheel4_omniwheel_tyre_v1_11, origin xyz=0.0384102 0.0124802 0.0065 rpy=1.5708 -0.971379 -2.82743, axis 0 0 1, limit effort=5 velocity=10
- added joint wheel_3k: type continuous, parent wheel4_shaft_holder_v2, child wheel4_omniwheel_tyre_v1, origin xyz=-0.0403869 2.57317e-17 0.0255 rpy=1.5708 0.992087 -3.14159, axis 0 0 1, limit effort=5 velocity=10
- added joint wheel_3l: type continuous, parent wheel4_shaft_holder_v2, child wheel4_omniwheel_tyre_v1_2, origin xyz=-0.0326737 0.0237388 0.0255 rpy=-1.5708 -0.508017 -0.628319, axis 0 0 1, limit effort=5 velocity=10
- added joint wheel_3m: type continuous, parent wheel4_shaft_holder_v2, child wheel4_omniwheel_tyre_v1_3, origin xyz=-0.0124802 0.0384102 0.0255 rpy=-1.5708 -0.0501607 -1.25664, axis 0 0 1, limit effort=5 velocity=10
- added joint wheel_3n: type continuous, parent wheel4_shaft_holder_v2, child wheel4_omniwheel_tyre_v1_4, origin xyz=0.0124802 0.0384102 0.0255 rpy=1.5708 -0.0501607 -1.88496, axis 0 0 1, limit effort=5 velocity=10
- added joint wheel_3o: type continuous, parent wheel4_shaft_holder_v2, child wheel4_omniwheel_tyre_v1_5, origin xyz=0.0326737 0.0237388 0.0255 rpy=1.5708 -0.508017 -2.51327, axis 0 0 1, limit effort=5 velocity=10
- added joint wheel_3p: type continuous, parent wheel4_shaft_holder_v2, child wheel4_omniwheel_tyre_v1_6, origin xyz=0.0403869 2.92012e-17 0.0255 rpy=1.5708 0.992087 -3.14159, axis 0 0 1, limit effort=5 velocity=10
- added joint wheel_3q: type continuous, parent wheel4_shaft_holder_v2, child wheel4_omniwheel_tyre_v1_7, origin xyz=0.0326737 -0.0237388 0.0255 rpy=-1.5708 -0.508017 -0.628319, axis 0 0 1, limit effort=5 velocity=10
- added joint wheel_3r: type continuous, parent wheel4_shaft_holder_v2, child wheel4_omniwheel_tyre_v1_8, origin xyz=0.0124802 -0.0384102 0.0255 rpy=-1.5708 -0.614515 -1.25664, axis 0 0 1, limit effort=5 velocity=10
- added joint wheel_3s: type continuous, parent wheel4_shaft_holder_v2, child wheel4_omniwheel_tyre_v1_9, origin xyz=-0.0124802 -0.0384102 0.0255 rpy=1.5708 -0.0501607 -1.88496, axis 0 0 1, limit effort=5 velocity=10
- added joint wheel_3t: type continuous, parent wheel4_shaft_holder_v2, child wheel4_omniwheel_tyre_v1_10, origin xyz=-0.0326737 -0.0237388 0.0255 rpy=1.5708 -0.508017 -2.51327, axis 0 0 1, limit effort=5 velocity=10
- added joint wheel_4a: type continuous, parent wheel4_shaft_holder_v2_3, child wheel4_omniwheel_tyre_v1_60, origin xyz=0.0384102 -0.0124802 0.0065 rpy=-1.25664 1.5708 0, axis 0 0 1, limit effort=5 velocity=10
- added joint wheel_4b: type continuous, parent wheel4_shaft_holder_v2_3, child wheel4_omniwheel_tyre_v1_59, origin xyz=0.0237388 -0.0326737 0.0065 rpy=-0.628319 1.5708 0, axis 0 0 1, limit effort=5 velocity=10
- added joint wheel_4c: type continuous, parent wheel4_shaft_holder_v2_3, child wheel4_omniwheel_tyre_v1_58, origin xyz=8.67362e-18 -0.0403869 0.0065 rpy=-3.38788e-16 1.5708 0, axis 0 0 1, limit effort=5 velocity=10
- added joint wheel_4d: type continuous, parent wheel4_shaft_holder_v2_3, child wheel4_omniwheel_tyre_v1_57, origin xyz=-0.0237388 -0.0326737 0.0065 rpy=-1.5708 1.54071 -2.19911, axis 0 0 1, limit effort=5 velocity=10
- added joint wheel_4e: type continuous, parent wheel4_shaft_holder_v2_3, child wheel4_omniwheel_tyre_v1_56, origin xyz=-0.0384102 -0.0124802 0.0065 rpy=1.25664 1.5708 0, axis 0 0 1, limit effort=5 velocity=10
- added joint wheel_4f: type continuous, parent wheel4_shaft_holder_v2_3, child wheel4_omniwheel_tyre_v1_55, origin xyz=-0.0384102 0.0124802 0.0065 rpy=-1.5708 1.54666 -0.314159, axis 0 0 1, limit effort=5 velocity=10
- added joint wheel_4g: type continuous, parent wheel4_shaft_holder_v2_3, child wheel4_omniwheel_tyre_v1_54, origin xyz=-0.0237388 0.0326737 0.0065 rpy=-0.628319 1.5708 0, axis 0 0 1, limit effort=5 velocity=10
- added joint wheel_4h: type continuous, parent wheel4_shaft_holder_v2_3, child wheel4_omniwheel_tyre_v1_53, origin xyz=3.46945e-18 0.0403869 0.0065 rpy=-4.44089e-16 1.5708 0, axis 0 0 1, limit effort=5 velocity=10
- added joint wheel_4i: type continuous, parent wheel4_shaft_holder_v2_3, child wheel4_omniwheel_tyre_v1_52, origin xyz=0.0237388 0.0326737 0.0065 rpy=0.628319 1.5708 0, axis 0 0 1, limit effort=5 velocity=10
- added joint wheel_4j: type continuous, parent wheel4_shaft_holder_v2_3, child wheel4_omniwheel_tyre_v1_51, origin xyz=0.0384102 0.0124802 0.0065 rpy=-1.88496 1.5708 0, axis 0 0 1, limit effort=5 velocity=10
- added joint wheel_4k: type continuous, parent wheel4_shaft_holder_v2_3, child wheel4_omniwheel_tyre_v1_41, origin xyz=-0.0403869 1.74979e-17 0.0255 rpy=-1.5708 1.5708 0, axis 0 0 1, limit effort=5 velocity=10
- added joint wheel_4l: type continuous, parent wheel4_shaft_holder_v2_3, child wheel4_omniwheel_tyre_v1_42, origin xyz=-0.0326737 0.0237388 0.0255 rpy=-0.942478 1.5708 0, axis 0 0 1, limit effort=5 velocity=10
- added joint wheel_4m: type continuous, parent wheel4_shaft_holder_v2_3, child wheel4_omniwheel_tyre_v1_43, origin xyz=-0.0124802 0.0384102 0.0255 rpy=-0.314159 1.5708 0, axis 0 0 1, limit effort=5 velocity=10
- added joint wheel_4n: type continuous, parent wheel4_shaft_holder_v2_3, child wheel4_omniwheel_tyre_v1_44, origin xyz=0.0124802 0.0384102 0.0255 rpy=-2.82743 1.5708 0, axis 0 0 1, limit effort=5 velocity=10
- added joint wheel_4o: type continuous, parent wheel4_shaft_holder_v2_3, child wheel4_omniwheel_tyre_v1_45, origin xyz=0.0326737 0.0237388 0.0255 rpy=-2.19911 1.5708 0, axis 0 0 1, limit effort=5 velocity=10
- added joint wheel_4p: type continuous, parent wheel4_shaft_holder_v2_3, child wheel4_omniwheel_tyre_v1_46, origin xyz=0.0403869 2.44368e-17 0.0255 rpy=-1.5708 1.5708 0, axis 0 0 1, limit effort=5 velocity=10
- added joint wheel_4q: type continuous, parent wheel4_shaft_holder_v2_3, child wheel4_omniwheel_tyre_v1_47, origin xyz=0.0326737 -0.0237388 0.0255 rpy=-0.942478 1.5708 0, axis 0 0 1, limit effort=5 velocity=10
- added joint wheel_4r: type continuous, parent wheel4_shaft_holder_v2_3, child wheel4_omniwheel_tyre_v1_48, origin xyz=0.0124802 -0.0384102 0.0255 rpy=-1.5708 1.00644 -1.25664, axis 0 0 1, limit effort=5 velocity=10
- added joint wheel_4s: type continuous, parent wheel4_shaft_holder_v2_3, child wheel4_omniwheel_tyre_v1_49, origin xyz=-0.0124802 -0.0384102 0.0255 rpy=-2.82743 1.5708 0, axis 0 0 1, limit effort=5 velocity=10
- added joint wheel_4t: type continuous, parent wheel4_shaft_holder_v2_3, child wheel4_omniwheel_tyre_v1_50, origin xyz=-0.0326737 -0.0237388 0.0255 rpy=-2.19911 1.5708 0, axis 0 0 1, limit effort=5 velocity=10
- added joint wheel_a: type continuous, parent wheel4_shaft_holder_v2_2, child wheel4_omniwheel_tyre_v1_40, origin xyz=0.0384102 -0.0124802 0.0065 rpy=-1.25664 1.5708 0, axis 0 0 1, limit effort=5 velocity=10
- added joint wheel_b: type continuous, parent wheel4_shaft_holder_v2_2, child wheel4_omniwheel_tyre_v1_39, origin xyz=0.0237388 -0.0326737 0.0065 rpy=1.5708 -0.210366 2.19911, axis 0 0 1, limit effort=5 velocity=10
- added joint wheel_c: type continuous, parent wheel4_shaft_holder_v2_2, child wheel4_omniwheel_tyre_v1_38, origin xyz=0 -0.0403869 0.0065 rpy=1.5708 6.10623e-16 1.5708, axis 0 0 1, limit effort=5 velocity=10
- added joint wheel_d: type continuous, parent wheel4_shaft_holder_v2_2, child wheel4_omniwheel_tyre_v1_37, origin xyz=-0.0237388 -0.0326737 0.0065 rpy=1.5708 -0.180277 0.942478, axis 0 0 1, limit effort=5 velocity=10
- added joint wheel_e: type continuous, parent wheel4_shaft_holder_v2_2, child wheel4_omniwheel_tyre_v1_36, origin xyz=-0.0384102 -0.0124802 0.0065 rpy=1.5708 -0.971379 0.314159, axis 0 0 1, limit effort=5 velocity=10
- added joint wheel_f: type continuous, parent wheel4_shaft_holder_v2_2, child wheel4_omniwheel_tyre_v1_35, origin xyz=-0.0384102 0.0124802 0.0065 rpy=1.5708 -0.947246 2.82743, axis 0 0 1, limit effort=5 velocity=10
- added joint wheel_g: type continuous, parent wheel4_shaft_holder_v2_2, child wheel4_omniwheel_tyre_v1_34, origin xyz=-0.0237388 0.0326737 0.0065 rpy=1.5708 -0.210366 2.19911, axis 0 0 1, limit effort=5 velocity=10
- added joint wheel_h: type continuous, parent wheel4_shaft_holder_v2_2, child wheel4_omniwheel_tyre_v1_33, origin xyz=-1.73472e-18 0.0403869 0.0065 rpy=-4.44089e-16 1.5708 0, axis 0 0 1, limit effort=5 velocity=10
- added joint wheel_i: type continuous, parent wheel4_shaft_holder_v2_2, child wheel4_omniwheel_tyre_v1_32, origin xyz=0.0237388 0.0326737 0.0065 rpy=1.5708 -0.210366 0.942478, axis 0 0 1, limit effort=5 velocity=10
- added joint wheel_j: type continuous, parent wheel4_shaft_holder_v2_2, child wheel4_omniwheel_tyre_v1_31, origin xyz=0.0384102 0.0124802 0.0065 rpy=-1.5708 -0.971379 0.314159, axis 0 0 1, limit effort=5 velocity=10
- added joint wheel_k: type continuous, parent wheel4_shaft_holder_v2_2, child wheel4_omniwheel_tyre_v1_21, origin xyz=-0.0403869 -6.36065e-18 0.0255 rpy=1.5708 0.992087 -3.14159, axis 0 0 1, limit effort=5 velocity=10
- added joint wheel_l: type continuous, parent wheel4_shaft_holder_v2_2, child wheel4_omniwheel_tyre_v1_22, origin xyz=-0.0326737 0.0237388 0.0255 rpy=1.5708 -0.508017 2.51327, axis 0 0 1, limit effort=5 velocity=10
- added joint wheel_m: type continuous, parent wheel4_shaft_holder_v2_2, child wheel4_omniwheel_tyre_v1_23, origin xyz=-0.0124802 0.0384102 0.0255 rpy=1.5708 -0.0501607 1.88496, axis 0 0 1, limit effort=5 velocity=10
- added joint wheel_n: type continuous, parent wheel4_shaft_holder_v2_2, child wheel4_omniwheel_tyre_v1_24, origin xyz=0.0124802 0.0384102 0.0255 rpy=-1.5708 -0.0501607 1.25664, axis 0 0 1, limit effort=5 velocity=10
- added joint wheel_o: type continuous, parent wheel4_shaft_holder_v2_2, child wheel4_omniwheel_tyre_v1_25, origin xyz=0.0326737 0.0237388 0.0255 rpy=-1.5708 -0.508017 0.628319, axis 0 0 1, limit effort=5 velocity=10
- added joint wheel_p: type continuous, parent wheel4_shaft_holder_v2_2, child wheel4_omniwheel_tyre_v1_26, origin xyz=0.0403869 -6.36065e-18 0.0255 rpy=1.5708 0.992087 -3.14159, axis 0 0 1, limit effort=5 velocity=10
- added joint wheel_q: type continuous, parent wheel4_shaft_holder_v2_2, child wheel4_omniwheel_tyre_v1_27, origin xyz=0.0326737 -0.0237388 0.0255 rpy=1.5708 -0.508017 2.51327, axis 0 0 1, limit effort=5 velocity=10
- added joint wheel_r: type continuous, parent wheel4_shaft_holder_v2_2, child wheel4_omniwheel_tyre_v1_28, origin xyz=0.0124802 -0.0384102 0.0255 rpy=1.5708 0.514194 1.88496, axis 0 0 1, limit effort=5 velocity=10
- added joint wheel_s: type continuous, parent wheel4_shaft_holder_v2_2, child wheel4_omniwheel_tyre_v1_29, origin xyz=-0.0124802 -0.0384102 0.0255 rpy=-1.5708 -0.0501607 1.25664, axis 0 0 1, limit effort=5 velocity=10
- added joint wheel_t: type continuous, parent wheel4_shaft_holder_v2_2, child wheel4_omniwheel_tyre_v1_30, origin xyz=-0.0326737 -0.0237388 0.0255 rpy=-1.5708 -0.508017 0.628319, axis 0 0 1, limit effort=5 velocity=10
- joint motorA_frame: parent wheel_4_2 -> wheel4_shaft_holder_v2_2
- joint motorB_frame: parent wheel_4_4 -> wheel4_shaft_holder_v2_4
- joint motorC_frame: parent wheel_4 -> wheel4_shaft_holder_v2
- joint motorD_frame: parent wheel_4_3 -> wheel4_shaft_holder_v2_3
- joint wheel_motorA: child wheel_4_2 -> wheel4_shaft_holder_v2_2
- joint wheel_motorB: child wheel_4_4 -> wheel4_shaft_holder_v2_4
- joint wheel_motorC: child wheel_4 -> wheel4_shaft_holder_v2
- joint wheel_motorD: child wheel_4_3 -> wheel4_shaft_holder_v2_3
