Commit message: model orientation changes and rviz view changes.

File: ros_gz_omni_description/models/omni_drive/robot.urdf (robot description, URDF)
Before this commit: robot omni_drive, 90 links, 89 joints
Joints:
- joint motorA_frame: origin xyz=0 3.37024e-19 0 rpy=3.14159 -1.12014e-59 -1.5708 -> xyz=0 1.96262e-17 1.38778e-17 rpy=3.14159 -0 -1.5708
- joint motorB_frame: origin xyz=-1.73472e-18 3.37024e-19 0 rpy=3.14159 -5.60071e-60 -1.5708 -> xyz=0 1.38778e-17 1.38778e-17 rpy=3.14159 -0 -1.5708
- joint motorC_frame: origin xyz=0 3.37024e-19 0 rpy=-2.36658e-30 1.63005e-32 -1.5708 -> xyz=0 1.14967e-17 1.38778e-17 rpy=-2.36658e-30 -0 -1.5708
- joint motorD_frame: origin xyz=0 -1.53081e-19 0 rpy=3.14159 -5.04871e-29 3.14159 -> xyz=1.73472e-18 6.93889e-18 -1.38778e-17 rpy=3.14159 -5.04871e-29 3.14159
- joint omni_drive_frame: origin xyz=-0.00053136 -0.000526049 0.025 rpy=0 -0 0.785398 -> xyz=-0.000747701 3.75549e-06 0.025 rpy=0 -0 0
- joint wheel_2c: origin xyz=1.21431e-17 -0.0403869 0.0065 rpy=-3.14159 -1.5708 0 -> xyz=1.73472e-18 -0.0403869 0.0065 rpy=-3.14159 -1.5708 0
- joint wheel_2k: origin xyz=-0.0403869 -2.71773e-17 0.0255 rpy=1.5708 0.992087 3.14159 -> xyz=-0.0403869 -2.77556e-17 0.0255 rpy=1.5708 0.992087 3.14159
- joint wheel_2p: origin xyz=0.0403869 2.83338e-17 0.0255 rpy=1.5708 0.992087 3.14159 -> xyz=0.0403869 5.55112e-17 0.0255 rpy=1.5708 0.992087 3.14159
- joint wheel_3c: origin xyz=-3.46945e-18 -0.0403869 0.0065 rpy=-1.5708 -6.10623e-16 -1.5708 -> xyz=-1.73472e-18 -0.0403869 0.0065 rpy=-1.5708 -6.66134e-16 -1.5708
- joint wheel_3h: origin xyz=0 0.0403869 0.0065 rpy=-4.44089e-16 1.5708 0 -> xyz=1.73472e-18 0.0403869 0.0065 rpy=-4.44089e-16 1.5708 0
- joint wheel_3k: origin xyz=-0.0403869 2.57317e-17 0.0255 rpy=1.5708 0.992087 -3.14159 -> xyz=-0.0403869 1.14967e-17 0.0255 rpy=1.5708 0.992087 -3.14159
- joint wheel_3p: origin xyz=0.0403869 2.92012e-17 0.0255 rpy=1.5708 0.992087 -3.14159 -> xyz=0.0403869 2.53745e-17 0.0255 rpy=1.5708 0.992087 -3.14159
- joint wheel_4c: origin xyz=8.67362e-18 -0.0403869 0.0065 rpy=-3.38788e-16 1.5708 0 -> xyz=0 -0.0403869 0.0065 rpy=-3.38788e-16 1.5708 0
- joint wheel_4h: origin xyz=3.46945e-18 0.0403869 0.0065 rpy=-4.44089e-16 1.5708 0 -> xyz=1.21431e-17 0.0403869 0.0065 rpy=-4.44089e-16 1.5708 0
- joint wheel_4k: origin xyz=-0.0403869 1.74979e-17 0.0255 rpy=-1.5708 1.5708 0 -> xyz=-0.0403869 8.79956e-32 0.0255 rpy=-1.5708 1.5708 0
- joint wheel_4p: origin xyz=0.0403869 2.44368e-17 0.0255 rpy=-1.5708 1.5708 0 -> xyz=0.0403869 4.16334e-17 0.0255 rpy=-1.5708 1.5708 0
- joint wheel_c: origin xyz=0 -0.0403869 0.0065 rpy=1.5708 6.10623e-16 1.5708 -> xyz=3.46945e-18 -0.0403869 0.0065 rpy=1.5708 6.66134e-16 1.5708
- joint wheel_k: origin xyz=-0.0403869 -6.36065e-18 0.0255 rpy=1.5708 0.992087 -3.14159 -> xyz=-0.0403869 1.96262e-17 0.0255 rpy=1.5708 0.992087 -3.14159
- joint wheel_motorA: origin xyz=6.36065e-18 0.105 0.0125 rpy=-1.5708 -1.5708 0 -> xyz=0.0742462 0.0742462 0.0125 rpy=-2.35619 -1.5708 0
- joint wheel_motorB: origin xyz=0.105 -6.36065e-18 0.0125 rpy=3.14159 -1.5708 0 -> xyz=0.0742462 -0.0742462 0.0125 rpy=2.35619 -1.5708 0
- joint wheel_motorC: origin xyz=4.91505e-18 -0.105 0.0125 rpy=1.5708 -1.5708 0 -> xyz=-0.0742462 -0.0742462 0.0125 rpy=0.785398 -1.5708 0
- joint wheel_motorD: origin xyz=-0.105 -1.74334e-17 0.0125 rpy=-1.63015e-15 -1.5708 0 -> xyz=-0.0742462 0.0742462 0.0125 rpy=-0.785398 -1.5708 0
- joint wheel_p: origin xyz=0.0403869 -6.36065e-18 0.0255 rpy=1.5708 0.992087 -3.14159 -> xyz=0.0403869 3.35039e-17 0.0255 rpy=1.5708 0.992087 -3.14159
